Commit message: re-organized

File: project_ws/src/my_simulation/my_simulation/models/urdf/bocbot.urdf (robot description, URDF)
Before this commit: robot epuck, 6 links, 5 joints
Links:
- link chassis: geometry collision mesh filename=/home/romi/project_ws/src/my_simulation/my_simulation/meshe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; visual mesh filename=/home/romi/project_ws/src/my_simulation/my_simulation/meshe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
- link left_wheel: geometry collision mesh filename=/home/romi/project_ws/src/my_simulation/my_simulation/meshe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; visual mesh filename=/home/romi/project_ws/src/my_simulation/my_simulation/meshe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
- link right_wheel: geometry collision mesh filename=/home/romi/project_ws/src/my_simulation/my_simulation/meshe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; visual mesh filename=/home/romi/project_ws/src/my_simulation/my_simulation/meshe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
